File: ebox-pinheader/ebox-pinheader.sch (KiCad schematic (older format))
At the start: 2 parts, among them J1 xconch_pinheader_2x40, J2 xconch_pinsocket_2x40

Commit message: ebox, modify some lib
Connections:
- net labels added: NC0, NC1, NC10, NC11, NC12, NC13, NC14, NC15, NC16, NC17, NC18, NC19, NC2, NC20, NC21, NC22, NC23, NC24, NC25, NC26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
- net labels removed: BAT-
- wire segments 135 -> 120
