File: ebox-pinheader/ebox-pinheader.kicad_pcb (KiCad board)
At the start: 2 copper layers, 2 parts, among them J1 xconch_pinheader_2x40, J2 xconch_pinsocket_2x40

Commit message: add i2c eerprom
Other:
- board outline added: 125 x 75 mm
